File: hub_ctrl.sch (KiCad schematic (older format))
At the start: 1 part

Commit message: preliminary schematic using discrete logic chips
Parts:
- J3: renamed from J?; footprint (none) -> Pin_Headers:Pin_Header_Straight_1x08_Pitch2.54mm
Connections:
- net switch_store: now reaches J3.8 (Pin_8)
Changed lines of the file:
@@
 LIBS:contrib
 LIBS:valves
+LIBS:74cbtlv3245
+LIBS:abb
+LIBS:tca9546a
 LIBS:flexibleaudiohub-cache
 EELAYER 25 0
@@
 $Descr A4 11693 8268
 encoding utf-8
-Sheet 5 9
+Sheet 4 10
 Title ""
 Date ""
@@
 only one power port will be required once a chip is chosen (3v3 most likely)
 $Comp
-L Conn_01x08 J?
+L Conn_01x08 J3
 U 1 1 5ADA6C91
 P 3700 2200
-F 0 "J?" H 3700 2600 50  0000 C CNN
+F 0 "J3" H 3700 2600 50  0000 C CNN
 F 1 "Conn_01x08" H 3700 1700 50  0000 C CNN
-F 2 "" H 3700 2200 50  0001 C CNN
+F 2 "Pin_Headers:Pin_Header_Straight_1x08_Pitch2.54mm" H 3700 2200 50  0001 C CNN
 F 3 "" H 3700 2200 50  0001 C CNN
 	1    3700 2200
@@
 Wire Wire Line
 	3100 2500 3500 2500
+Text HLabel 3100 2600 0    60   Output ~ 0
+switch_store
+Wire Wire Line
+	3500 2600 3100 2600
 $EndSCHEMATC
