File: bus_sw_2x2.sch (KiCad schematic (older format))
At the start: 32 parts, among them U4 74CBTLV3245, U5 74CBTLV3245, U6 74CBTLV3245, U7 74CBTLV3245

Commit message: finished layout
Parts:
- added C14, C15: C_Small, Capacitors_SMD:C_0805_HandSoldering, symbol C_Small
- added R45, R46, R47, R48, R49, R50, R51, R52, R53, R54, R55, R9: R_Small, Resistors_SMD:R_0805_HandSoldering, symbol R_Small
- added U10, U11: 74CBTLV3245, Housings_SSOP:TSSOP-20_4.4x6.5mm_Pitch0.65mm, symbol 74CBTLV3245
Connections:
- net labels added: i2sin02, i2sout02, lrclk02, mclk02, sclk02, sw_00_01, sw_02_03
- wire segments 124 -> 178
Other:
- note added: "replace these resistors with an 0805 footprint that is shorted?\n(i.e. 0R pre-installed, cut track if needed)"
- note removed: "this is not a full crossbar layout, but should be sufficient to test \n(up to 2 inputs and up to 2 outputs)"
- moved on the sheet: C4, C5, C6, C7, R21, R22, R23, R24, R25, R26, R27, R28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
