File: flexibleaudiohub.sch (KiCad schematic (older format))
At the start: 0 parts

Commit message: preliminary schematic using discrete logic chips
Parts:
- added C1: C_Small, Capacitors_SMD:C_0805_HandSoldering, symbol C_Small
- added R1, R2: 3k9, Resistors_SMD:R_0805_HandSoldering, symbol R_Small
- added U1: AT24CS32-SSHM, Housings_SOIC:SOIC-8_3.9x4.9mm_Pitch1.27mm, symbol AT24CS32-SSHM
Connections:
- net +3V3: now also C1.1, R1.1, R2.1, U1.8 (VCC)
- net GND: now also C1.2, U1.1 (A0), U1.2 (A1), U1.3 (A2), U1.4 (GND), U1.7 (WP)
- new net hat_id_scl: R1.2, U1.6 (SCL)
- new net hat_id_sda: R2.2, U1.5 (SDA)
Other:
- note added: "CAT24C32 is recommended in HAT design guide\nAT24C32, AT24CS32, and others are equivalent"
- note added: "HAT ID EEPROM"
Changed lines of the file:
@@
 LIBS:contrib
 LIBS:valves
+LIBS:74cbtlv3245
+LIBS:abb
+LIBS:tca9546a
 LIBS:flexibleaudiohub-cache
 EELAYER 25 0
@@
 $Descr A4 11693 8268
 encoding utf-8
-Sheet 1 9
+Sheet 1 10
 Title ""
 Date ""
@@
 F9 "5v" B L 1050 2150 60
 F10 "3v3" O L 1050 2250 60
+F11 "ID_SDA" B R 1900 2400 60
+F12 "ID_SCL" B R 1900 2500 60
 $EndSheet
 $Sheet
@@
 $EndSheet
 $Comp
-L GND #PWR?
+L GND #PWR01
 U 1 1 5AD775EA
 P 950 3300
-F 0 "#PWR?" H 950 3050 50  0001 C CNN
+F 0 "#PWR01" H 950 3050 50  0001 C CNN
 F 1 "GND" H 950 3150 50  0000 C CNN
 F 2 "" H 950 3300 50  0001 C CNN
@@
 $EndComp
 $Comp
-L +5V #PWR?
+L +5V #PWR02
 U 1 1 5AD776BD
 P 950 2100
-F 0 "#PWR?" H 950 1950 50  0001 C CNN
+F 0 "#PWR02" H 950 1950 50  0001 C CNN
 F 1 "+5V" H 950 2240 50  0000 C CNN
 F 2 "" H 950 2100 50  0001 C CNN
@@
 $EndComp
 $Comp
-L +12V #PWR?
+L +12V #PWR03
 U 1 1 5AD77CF2
 P 1700 3900
-F 0 "#PWR?" H 1700 3750 50  0001 C CNN
+F 0 "#PWR03" H 1700 3750 50  0001 C CNN
 F 1 "+12V" H 1700 4040 50  0000 C CNN
 F 2 "" H 1700 3900 50  0001 C CNN
@@
 $EndComp
 $Comp
-L +5V #PWR?
+L +5V #PWR04
 U 1 1 5AD77E86
 P 1950 3900
-F 0 "#PWR?" H 1950 3750 50  0001 C CNN
+F 0 "#PWR04" H 1950 3750 50  0001 C CNN
 F 1 "+5V" H 1950 4040 50  0000 C CNN
 F 2 "" H 1950 3900 50  0001 C CNN
@@
 NoConn ~ 1050 2250
 $Comp
-L GND #PWR?
+L GND #PWR05
 U 1 1 5AD78117
 P 1700 5200
-F 0 "#PWR?" H 1700 4950 50  0001 C CNN
+F 0 "#PWR05" H 1700 4950 50  0001 C CNN
 F 1 "GND" H 1700 5050 50  0000 C CNN
 F 2 "" H 1700 5200 50  0001 C CNN
@@
 $EndComp
 $Comp
-L +3V3 #PWR?
+L +3V3 #PWR06
 U 1 1 5AD781EB
 P 2200 3900
-F 0 "#PWR?" H 2200 3750 50  0001 C CNN
+F 0 "#PWR06" H 2200 3750 50  0001 C CNN
 F 1 "+3V3" H 2200 4040 50  0000 C CNN
 F 2 "" H 2200 3900 50  0001 C CNN
@@
 F7 "switch_data" O R 4200 4100 60
 F8 "switch_clk" O R 4200 4200 60
+F9 "switch_store" O R 4200 4300 60
 $EndSheet
 $Sheet
@@
 F32 "LRclk_03" I R 7950 3450 60
 F33 "Mclk_03" I R 7950 3250 60
-$EndSheet
-$Comp
-L +3V3 #PWR?
+F34 "ctrl_store_clk" I R 7950 1100 60
+$EndSheet
+$Comp
+L +3V3 #PWR07
 U 1 1 5AD8FC7E
 P 6500 850
-F 0 "#PWR?" H 6500 700 50  0001 C CNN
+F 0 "#PWR07" H 6500 700 50  0001 C CNN
 F 1 "+3V3" H 6500 990 50  0000 C CNN
 F 2 "" H 6500 850 50  0001 C CNN
@@
 $EndComp
 $Comp
-L GND #PWR?
+L GND #PWR08
 U 1 1 5AD90A29
 P 6500 1050
-F 0 "#PWR?" H 6500 800 50  0001 C CNN
+F 0 "#PWR08" H 6500 800 50  0001 C CNN
 F 1 "GND" H 6500 900 50  0000 C CNN
 F 2 "" H 6500 1050 50  0001 C CNN
@@
 $EndComp
 $Comp
-L +12V #PWR?
+L +12V #PWR09
 U 1 1 5AD90F49
 P 5050 1450
-F 0 "#PWR?" H 5050 1300 50  0001 C CNN
+F 0 "#PWR09" H 5050 1300 50  0001 C CNN
 F 1 "+12V" H 5050 1590 50  0000 C CNN
 F 2 "" H 5050 1450 50  0001 C CNN
@@
 	5050 1500 5200 1500
 $Comp
-L GND #PWR?
+L GND #PWR010
 U 1 1 5AD93B9D
 P 5050 1650
-F 0 "#PWR?" H 5050 1400 50  0001 C CNN
+F 0 "#PWR010" H 5050 1400 50  0001 C CNN
 F 1 "GND" H 5050 1500 50  0000 C CNN
 F 2 "" H 5050 1650 50  0001 C CNN
@@
 	5050 1600 5050 1650
 $Comp
-L GND #PWR?
+L GND #PWR011
 U 1 1 5AD95AEF
 P 5550 3000
-F 0 "#PWR?" H 5550 2750 50  0001 C CNN
+F 0 "#PWR011" H 5550 2750 50  0001 C CNN
 F 1 "GND" H 5550 2850 50  0000 C CNN
 F 2 "" H 5550 3000 50  0001 C CNN
@@
 $EndComp
 $Comp
-L +12V #PWR?
+L +12V #PWR012
 U 1 1 5AD95CF8
 P 5550 2800
-F 0 "#PWR?" H 5550 2650 50  0001 C CNN
+F 0 "#PWR012" H 5550 2650 50  0001 C CNN
 F 1 "+12V" H 5550 2940 50  0000 C CNN
 F 2 "" H 5550 2800 50  0001 C CNN
@@
 	6250 3650 6600 3650
 $Comp
-L +12V #PWR?
+L +12V #PWR013
 U 1 1 5AD97A7D
 P 9150 2750
-F 0 "#PWR?" H 9150 2600 50  0001 C CNN
+F 0 "#PWR013" H 9150 2600 50  0001 C CNN
 F 1 "+12V" H 9150 2890 50  0000 C CNN
 F 2 "" H 9150 2750 50  0001 C CNN
@@
 $EndComp
 $Comp
-L GND #PWR?
+L GND #PWR014
 U 1 1 5AD97C95
 P 9150 2950
-F 0 "#PWR?" H 9150 2700 50  0001 C CNN
+F 0 "#PWR014" H 9150 2700 50  0001 C CNN
 F 1 "GND" H 9150 2800 50  0000 C CNN
 F 2 "" H 9150 2950 50  0001 C CNN
@@
 	8300 3650 7950 3650
 $Comp
-L +12V #PWR?
+L +12V #PWR015
 U 1 1 5AD996CC
 P 9150 1450
-F 0 "#PWR?" H 9150 1300 50  0001 C CNN
+F 0 "#PWR015" H 9150 1300 50  0001 C CNN
 F 1 "+12V" H 9150 1590 50  0000 C CNN
 F 2 "" H 9150 1450 50  0001 C CNN
@@
 $EndComp
 $Comp
-L GND #PWR?
+L GND #PWR016
 U 1 1 5AD998E3
 P 9150 1650
-F 0 "#PWR?" H 9150 1400 50  0001 C CNN
+F 0 "#PWR016" H 9150 1400 50  0001 C CNN
 F 1 "GND" H 9150 1500 50  0000 C CNN
 F 2 "" H 9150 1650 50  0001 C CNN
@@
 $EndSheet
 $Comp
-L +5V #PWR?
+L +5V #PWR017
 U 1 1 5ADB33CF
 P 2900 3950
-F 0 "#PWR?" H 2900 3800 50  0001 C CNN
+F 0 "#PWR017" H 2900 3800 50  0001 C CNN
 F 1 "+5V" H 2900 4090 50  0000 C CNN
 F 2 "" H 2900 3950 50  0001 C CNN
@@
 	2900 4100 3000 4100
 $Comp
-L +3V3 #PWR?
+L +3V3 #PWR018
 U 1 1 5ADB3734
 P 2700 3950
-F 0 "#PWR?" H 2700 3800 50  0001 C CNN
+F 0 "#PWR018" H 2700 3800 50  0001 C CNN
 F 1 "+3V3" H 2700 4090 50  0000 C CNN
 F 2 "" H 2700 3950 50  0001 C CNN
@@
 	2700 4200 3000 4200
 $Comp
-L GND #PWR?
+L GND #PWR019
 U 1 1 5ADB3FC3
 P 2450 4450
-F 0 "#PWR?" H 2450 4200 50  0001 C CNN
+F 0 "#PWR019" H 2450 4200 50  0001 C CNN
 F 1 "GND" H 2450 4300 50  0000 C CNN
 F 2 "" H 2450 4450 50  0001 C CNN
@@
 Wire Wire Line
 	2450 4300 2450 4450
+Wire Wire Line
+	7950 1100 8100 1100
+Text Label 8100 1100 0    60   ~ 0
+sw_ctrl_store
+Wire Wire Line
+	4200 4300 4450 4300
+Text Label 4450 4300 0    60   ~ 0
+sw_ctrl_store
+$Comp
+L AT24CS32-SSHM U1
+U 1 1 5ADCD07C
+P 4400 6350
+F 0 "U1" H 4200 6600 50  0000 C CNN
+F 1 "AT24CS32-SSHM" H 4700 6050 50  0000 C CNN
+F 2 "Housings_SOIC:SOIC-8_3.9x4.9mm_Pitch1.27mm" H 4400 6350 50  0001 C CIN
+F 3 "" H 4400 6350 50  0001 C CNN
+	1    4400 6350
+	1    0    0    -1
+$EndComp
+Text Notes 3150 5550 0    60   ~ 0
+HAT ID EEPROM
+$Comp
+L +3V3 #PWR020
+U 1 1 5ADCF723
+P 4400 5550
+F 0 "#PWR020" H 4400 5400 50  0001 C CNN
+F 1 "+3V3" H 4400 5690 50  0000 C CNN
+F 2 "" H 4400 5550 50  0001 C CNN
+F 3 "" H 4400 5550 50  0001 C CNN
+	1    4400 5550
+	1    0    0    -1
+$EndComp
+Wire Wire Line
+	4400 5550 4400 6000
+$Comp
+L C_Small C1
+U 1 1 5ADD0A63
+P 4650 5950
+F 0 "C1" H 4660 6020 50  0000 L CNN
+F 1 "C_Small" H 4660 5870 50  0000 L CNN
+F 2 "Capacitors_SMD:C_0805_HandSoldering" H 4650 5950 50  0001 C CNN
+F 3 "" H 4650 5950 50  0001 C CNN
+	1    4650 5950
+	0    -1   -1   0
+$EndComp
+Wire Wire Line
+	4550 5950 4400 5950
+Connection ~ 4400 5950
+$Comp
+L GND #PWR021
+U 1 1 5ADD13E2
+P 4900 6000
+F 0 "#PWR021" H 4900 5750 50  0001 C CNN
+F 1 "GND" H 4900 5850 50  0000 C CNN
+F 2 "" H 4900 6000 50  0001 C CNN
+F 3 "" H 4900 6000 50  0001 C CNN
+	1    4900 6000
+	1    0    0    -1
+$EndComp
+Wire Wire Line
+	4900 5950 4900 6000
+$Comp
+L GND #PWR022
+U 1 1 5ADD177E
+P 4400 6900
+F 0 "#PWR022" H 4400 6650 50  0001 C CNN
+F 1 "GND" H 4400 6750 50  0000 C CNN
+F 2 "" H 4400 6900 50  0001 C CNN
+F 3 "" H 4400 6900 50  0001 C CNN
+	1    4400 6900
+	1    0    0    -1
+$EndComp
+Wire Wire Line
+	4400 6750 4400 6900
+Wire Wire Line
+	4900 5950 4750 5950
+Text Label 1900 2400 0    60   ~ 0
+hat_id_sda
+Text Label 1900 2500 0    60   ~ 0
+hat_id_scl
+Text Label 6000 6250 0    60   ~ 0
+hat_id_sda
+Text Label 6000 6400 0    60   ~ 0
+hat_id_scl
+Wire Wire Line
+	4000 6200 3900 6200
+Wire Wire Line
+	3900 6200 3900 6800
+Wire Wire Line
+	3900 6800 4400 6800
+Connection ~ 4400 6800
+Wire Wire Line
+	4000 6300 3900 6300
+Connection ~ 3900 6300
+Wire Wire Line
+	4000 6400 3900 6400
+Connection ~ 3900 6400
+Wire Wire Line
+	4000 6550 3900 6550
+Connection ~ 3900 6550
+$Comp
+L R_Small R2
+U 1 1 5ADD4E9A
+P 5800 6050
+F 0 "R2" H 5830 6070 50  0000 L CNN
+F 1 "3k9" H 5830 6010 50  0000 L CNN
+F 2 "Resistors_SMD:R_0805_HandSoldering" H 5800 6050 50  0001 C CNN
+F 3 "" H 5800 6050 50  0001 C CNN
+	1    5800 6050
+	1    0    0    -1
+$EndComp
+$Comp
+L R_Small R1
+U 1 1 5ADD510C
+P 5550 6050
+F 0 "R1" H 5580 6070 50  0000 L CNN
+F 1 "3k9" H 5580 6010 50  0000 L CNN
+F 2 "Resistors_SMD:R_0805_HandSoldering" H 5550 6050 50  0001 C CNN
+F 3 "" H 5550 6050 50  0001 C CNN
+	1    5550 6050
+	1    0    0    -1
+$EndComp
+Wire Wire Line
+	6000 6250 4800 6250
+Wire Wire Line
+	4800 6400 6000 6400
+Wire Wire Line
+	4400 5600 5800 5600
+Wire Wire Line
+	5800 5600 5800 5950
+Connection ~ 4400 5600
+Wire Wire Line
+	5550 5950 5550 5600
+Connection ~ 5550 5600
+Wire Wire Line
+	5550 6150 5550 6400
+Connection ~ 5550 6400
+Wire Wire Line
+	5800 6150 5800 6250
+Connection ~ 5800 6250
+Text Notes 3600 7300 0    60   ~ 0
+CAT24C32 is recommended in HAT design guide\nAT24C32, AT24CS32, and others are equivalent
 $EndSCHEMATC
