File: hub_power.sch (KiCad schematic (older format))
At the start: 8 parts

Commit message: preliminary schematic using discrete logic chips
Parts:
- added C12, C13: 10uF, Capacitors_THT:CP_Radial_D5.0mm_P2.00mm, symbol CP_Small
- C10, C11, C8, C9: renamed from C?; footprint (none) -> Capacitors_SMD:C_0805_HandSoldering
- D1: renamed from D?; footprint (none) -> Diodes_THT:D_5W_P10.16mm_Horizontal
- J7: renamed from J?; footprint (none) -> Resistors_SMD:R_0805_HandSoldering
- U8, U9: renamed from U?; footprint (none) -> TO_SOT_Packages_THT:TO-220_Vertical
Connections:
- net +12v: now also C12.1, C13.1
- net Gnd: now also C12.2, C13.2
Changed lines of the file:
@@
 LIBS:contrib
 LIBS:valves
+LIBS:74cbtlv3245
+LIBS:abb
+LIBS:tca9546a
 LIBS:flexibleaudiohub-cache
 EELAYER 25 0
@@
 $Descr A4 11693 8268
 encoding utf-8
-Sheet 4 9
+Sheet 10 10
 Title ""
 Date ""
@@
 +12v
 $Comp
-L Barrel_Jack J?
+L Barrel_Jack J7
 U 1 1 5AD75AA3
 P 3900 2800
-F 0 "J?" H 3900 3010 50  0000 C CNN
+F 0 "J7" H 3900 3010 50  0000 C CNN
 F 1 "Barrel_Jack" H 3900 2625 50  0000 C CNN
-F 2 "" H 3950 2760 50  0001 C CNN
+F 2 "Resistors_SMD:R_0805_HandSoldering" H 3950 2760 50  0001 C CNN
 F 3 "" H 3950 2760 50  0001 C CNN
 	1    3900 2800
@@
 	4200 2900 5900 2900
 $Comp
-L D D?
+L D D1
 U 1 1 5AD75B06
 P 4700 2800
-F 0 "D?" H 4700 2900 50  0000 C CNN
+F 0 "D1" H 4700 2900 50  0000 C CNN
 F 1 "D" H 4700 2700 50  0000 C CNN
-F 2 "" H 4700 2800 50  0001 C CNN
+F 2 "Diodes_THT:D_5W_P10.16mm_Horizontal" H 4700 2800 50  0001 C CNN
 F 3 "" H 4700 2800 50  0001 C CNN
 	1    4700 2800
@@
 	4850 2800 5900 2800
 $Comp
-L L7805 U?
+L L7805 U8
 U 1 1 5AD75B54
 P 5450 3900
-F 0 "U?" H 5300 4025 50  0000 C CNN
+F 0 "U8" H 5300 4025 50  0000 C CNN
 F 1 "L7805" H 5450 4025 50  0000 L CNN
-F 2 "" H 5475 3750 50  0001 L CIN
+F 2 "TO_SOT_Packages_THT:TO-220_Vertical" H 5475 3750 50  0001 L CIN
 F 3 "" H 5450 3850 50  0001 C CNN
 	1    5450 3900
 	1    0    0    -1
 $EndComp
-Text Notes 2400 3800 0    60   ~ 0
+Text Notes 3550 3550 0    60   ~ 0
 TODO: replace regs with buck conv.
 Text Label 5150 2800 0    60   ~ 0
 power_supp_12v
-Text Label 4500 3900 2    60   ~ 0
+Text Label 3650 3900 2    60   ~ 0
 power_supp_12v
 Wire Wire Line
-	4500 3900 5150 3900
-$Comp
-L C_Small C?
+	3650 3900 5150 3900
+$Comp
+L C_Small C8
 U 1 1 5AD75D36
 P 4950 4100
-F 0 "C?" H 4960 4170 50  0000 L CNN
+F 0 "C8" H 4960 4170 50  0000 L CNN
 F 1 "C_Small" H 4960 4020 50  0000 L CNN
-F 2 "" H 4950 4100 50  0001 C CNN
+F 2 "Capacitors_SMD:C_0805_HandSoldering" H 4950 4100 50  0001 C CNN
 F 3 "" H 4950 4100 50  0001 C CNN
 	1    4950 4100
@@
 	4950 4200 4950 4250
 Wire Wire Line
-	4950 4250 6800 4250
+	4550 4250 6800 4250
 Wire Wire Line
 	5450 4250 5450 4200
@@
 power_supp_gnd
 $Comp
-L C_Small C?
+L C_Small C11
 U 1 1 5AD75E0E
 P 5850 4100
-F 0 "C?" H 5860 4170 50  0000 L CNN
+F 0 "C11" H 5860 4170 50  0000 L CNN
 F 1 "C_Small" H 5860 4020 50  0000 L CNN
-F 2 "" H 5850 4100 50  0001 C CNN
+F 2 "Capacitors_SMD:C_0805_HandSoldering" H 5850 4100 50  0001 C CNN
 F 3 "" H 5850 4100 50  0001 C CNN
 	1    5850 4100
@@
 	5750 3900 6850 3900
 $Comp
-L LM1117-3.3 U?
+L LM1117-3.3 U9
 U 1 1 5AD75E6D
 P 5450 4750
-F 0 "U?" H 5300 4875 50  0000 C CNN
+F 0 "U9" H 5300 4875 50  0000 C CNN
 F 1 "LM1117-3.3" H 5450 4875 50  0000 L CNN
-F 2 "" H 5450 4750 50  0001 C CNN
+F 2 "TO_SOT_Packages_THT:TO-220_Vertical" H 5450 4750 50  0001 C CNN
 F 3 "" H 5450 4750 50  0001 C CNN
 	1    5450 4750
@@
 $EndComp
 $Comp
-L C_Small C?
+L C_Small C9
 U 1 1 5AD75ECA
 P 5000 4950
-F 0 "C?" H 5010 5020 50  0000 L CNN
+F 0 "C9" H 5010 5020 50  0000 L CNN
 F 1 "C_Small" H 5010 4870 50  0000 L CNN
-F 2 "" H 5000 4950 50  0001 C CNN
+F 2 "Capacitors_SMD:C_0805_HandSoldering" H 5000 4950 50  0001 C CNN
 F 3 "" H 5000 4950 50  0001 C CNN
 	1    5000 4950
@@
 $EndComp
 Wire Wire Line
-	4700 4750 5150 4750
-Wire Wire Line
-	4700 4750 4700 3900
-Connection ~ 4700 3900
+	4100 4750 5150 4750
 Wire Wire Line
 	5000 4850 5000 4750
@@
 	5000 5050 5000 5100
 Wire Wire Line
-	5000 5100 6300 5100
+	4450 5100 6300 5100
 Wire Wire Line
 	5450 5100 5450 5050
 $Comp
-L C_Small C?
+L C_Small C10
 U 1 1 5AD75F75
 P 5800 4950
-F 0 "C?" H 5810 5020 50  0000 L CNN
+F 0 "C10" H 5810 5020 50  0000 L CNN
 F 1 "C_Small" H 5810 4870 50  0000 L CNN
-F 2 "" H 5800 4950 50  0001 C CNN
+F 2 "Capacitors_SMD:C_0805_HandSoldering" H 5800 4950 50  0001 C CNN
 F 3 "" H 5800 4950 50  0001 C CNN
 	1    5800 4950
@@
 Text HLabel 6850 3900 2    60   Output ~ 0
 +5v
+$Comp
+L CP_Small C12
+U 1 1 5ADDA19C
+P 4450 4950
+F 0 "C12" H 4460 5020 50  0000 L CNN
+F 1 "10uF" H 4460 4870 50  0000 L CNN
+F 2 "Capacitors_THT:CP_Radial_D5.0mm_P2.00mm" H 4450 4950 50  0001 C CNN
+F 3 "" H 4450 4950 50  0001 C CNN
+	1    4450 4950
+	1    0    0    -1
+$EndComp
+Wire Wire Line
+	4450 4750 4450 4850
+Wire Wire Line
+	4450 5050 4450 5100
+Connection ~ 5000 5100
+$Comp
+L CP_Small C13
+U 1 1 5ADDA2E4
+P 4550 4100
+F 0 "C13" H 4560 4170 50  0000 L CNN
+F 1 "10uF" H 4560 4020 50  0000 L CNN
+F 2 "Capacitors_THT:CP_Radial_D5.0mm_P2.00mm" H 4550 4100 50  0001 C CNN
+F 3 "" H 4550 4100 50  0001 C CNN
+	1    4550 4100
+	1    0    0    -1
+$EndComp
+Wire Wire Line
+	4550 4200 4550 4250
+Connection ~ 4950 4250
+Wire Wire Line
+	4550 4000 4550 3900
+Connection ~ 4550 3900
+Wire Wire Line
+	4100 4750 4100 3900
+Connection ~ 4100 3900
+Connection ~ 4450 4750
 $EndSCHEMATC

Commit message: finished layout
Parts:
- J7: footprint Resistors_SMD:R_0805_HandSoldering -> Connectors:BARREL_JACK
Connections:
- net at J7.1: now also D1.2 (A)
- net at J7.3: no longer D1.2 (A)
Other:
- moved on the sheet: D1
Changed lines of the file:
@@
 Comment4 ""
 $EndDescr
-Text HLabel 5900 2800 2    60   Output ~ 0
+Text HLabel 5900 2700 2    60   Output ~ 0
 +12v
 $Comp
@@
 F 0 "J7" H 3900 3010 50  0000 C CNN
 F 1 "Barrel_Jack" H 3900 2625 50  0000 C CNN
-F 2 "Resistors_SMD:R_0805_HandSoldering" H 3950 2760 50  0001 C CNN
+F 2 "Connectors:BARREL_JACK" H 3950 2760 50  0001 C CNN
 F 3 "" H 3950 2760 50  0001 C CNN
 	1    3900 2800
@@
 L D D1
 U 1 1 5AD75B06
-P 4700 2800
-F 0 "D1" H 4700 2900 50  0000 C CNN
-F 1 "D" H 4700 2700 50  0000 C CNN
-F 2 "Diodes_THT:D_5W_P10.16mm_Horizontal" H 4700 2800 50  0001 C CNN
-F 3 "" H 4700 2800 50  0001 C CNN
-	1    4700 2800
+P 4700 2700
+F 0 "D1" H 4700 2800 50  0000 C CNN
+F 1 "D" H 4700 2600 50  0000 C CNN
+F 2 "Diodes_THT:D_5W_P10.16mm_Horizontal" H 4700 2700 50  0001 C CNN
+F 3 "" H 4700 2700 50  0001 C CNN
+	1    4700 2700
 	-1   0    0    1
 $EndComp
 Wire Wire Line
-	4200 2800 4550 2800
-Wire Wire Line
-	4850 2800 5900 2800
+	4850 2700 5900 2700
 $Comp
 L L7805 U8
@@
 Text Notes 3550 3550 0    60   ~ 0
 TODO: replace regs with buck conv.
-Text Label 5150 2800 0    60   ~ 0
+Text Label 5150 2700 0    60   ~ 0
 power_supp_12v
 Text Label 3650 3900 2    60   ~ 0
@@
 Connection ~ 4100 3900
 Connection ~ 4450 4750
+Wire Wire Line
+	4550 2700 4200 2700
 $EndSCHEMATC
